Commit message: add irobots

File: hector_quadrotor_description/urdf/irobot_base.urdf.xacro (robot description, xacro)
@@ -3,5 +3,6 @@
   <!-- <xacro:include filename="$(find hector_sensors_description)/urdf/sonar_sensor.urdf.xacro" /> -->
   <xacro:property name="pi" value="3.1415926535897931" />
-  <xacro:macro name="irobot_base_macro" params="name update_rate commandTopic odometryFrame robotBaseFrame">
+  <!-- <xacro:macro name="irobot_base_macro" params="name update_rate commandTopic odometryFrame robotBaseFrame"> -->
+  <xacro:macro name="irobot_base_macro" params="name">
     <link name="base">
       <inertial>
@@ -29,7 +30,5 @@
         <pose>0 0 0.047800 0 0 0</pose>
         <geometry>
-          <mesh>
-            <uri>model://create/meshes/create_body.dae</uri>
-          </mesh>
+            <mesh filename="package://hector_quadrotor_description/meshes/irobot/create_body.dae.dae"/>
         </geometry>
       </visual>
@@ -281,5 +280,6 @@
   <plugin name="differential_drive_controller" filename="libgazebo_ros_diff_drive.so">
     <alwaysOn>true</alwaysOn>
-    <updateRate>${update_rate}</updateRate>
+    <!-- <updateRate>${update_rate}</updateRate> -->
+    <updateRate>20</updateRate>
     <leftJoint>right_wheel</leftJoint>
     <rightJoint>left_wheel</rightJoint>
