Commit message: change kinect's postion on uav so that it will not see the propeller

File: hector_quadrotor_description/urdf/quadrotor_with_kinect_laser.urdf.xacro (robot description, xacro)
@@ -14,5 +14,5 @@
     <xacro:include filename="$(find hector_sensors_description)/urdf/kinect_camera.urdf.xacro" />
     <xacro:kinect_camera name="camera" parent="base_link">
-      <origin xyz="0.15 0.0 -0.06" rpy="0 0 0"/>
+      <origin xyz="0.18 0.0 -0.06" rpy="0 0 0"/>
     </xacro:kinect_camera>
 </robot>
