Commit message: add draw_circlr to control the uav fly a circle and add spinning lidar control to control the spinning lidar rotating

File: hector_quadrotor_description/urdf/quadrotor_downward_cam_spinning_lidar.urdf.xacro (robot description, xacro)
@@ -10,10 +10,10 @@
     <xacro:quadrotor_base_macro />
     <xacro:include filename="$(find hector_components_description)/urdf/spinning_hokuyo_utm30lx.urdf.xacro" />
-<!--     <xacro:spinning_hokuyo_utm30lx_macro name="spinning_hokuyo" parent="base_link" angle_deg="30" >
+    <xacro:spinning_hokuyo_utm30lx_macro name="spinning_hokuyo" parent="base_link" angle_deg="45" >
+      <origin xyz="0.0 0.0 -0.05" rpy="${M_PI} 0 0"/>
+    </xacro:spinning_hokuyo_utm30lx_macro>
+<!--     <xacro:spinning_hokuyo_utm30lx_lidar_mount_offset_macro name="spinning_hokuyo" parent="base_link" scan_topic_in_namespace="scan" angle_deg="45" >
       <origin xyz="0.0 0.0 -0.097" rpy="${M_PI} 0 0"/>
-    </xacro:spinning_hokuyo_utm30lx_macro> -->
-    <xacro:spinning_hokuyo_utm30lx_lidar_mount_offset_macro name="spinning_hokuyo_mount" parent="base_link" scan_topic_in_namespace="scan" angle_deg="45" >
-      <origin xyz="0.0 0.0 -0.097" rpy="${M_PI} 0 0"/>
-    </xacro:spinning_hokuyo_utm30lx_lidar_mount_offset_macro>
+    </xacro:spinning_hokuyo_utm30lx_lidar_mount_offset_macro> -->
     <!-- Downward facing camera -->
     <xacro:include filename="$(find hector_sensors_description)/urdf/generic_camera.urdf.xacro" />

File: hector_quadrotor_description/urdf/quadrotor_with_kinect_laser.urdf.xacro (robot description, xacro)
@@ -11,8 +11,13 @@
       <origin xyz="0.0 0.0 -0.097" rpy="${M_PI} 0 0"/>
     </xacro:hokuyo_utm30lx>
-    <!-- Kinect -->
+    <!-- Kinect forward-->
+<!--     <xacro:include filename="$(find hector_sensors_description)/urdf/kinect_camera.urdf.xacro" />
+    <xacro:kinect_camera name="camera" parent="base_link">
+      <origin xyz="0.18 0.0 -0.06" rpy="0 0 0"/>
+    </xacro:kinect_camera> -->
+    <!-- Kinect downward -->
     <xacro:include filename="$(find hector_sensors_description)/urdf/kinect_camera.urdf.xacro" />
     <xacro:kinect_camera name="camera" parent="base_link">
-      <origin xyz="0.18 0.0 -0.06" rpy="0 0 0"/>
+     <origin xyz="0.4 0.0 -0.0" rpy="0 ${M_PI/2} 0"/>
     </xacro:kinect_camera>
 </robot>

File: hector_quadrotor_description/urdf/quadrotor_with_wireless_receiver.urdf.xacro (robot description, xacro)
@@ -11,4 +11,9 @@
       <origin xyz="0.4 0.0 -0.0" rpy="0 ${M_PI/2} 0"/>
     </xacro:generic_camera> -->
+        <!-- Hokuyo UTM-30LX mounted upside down below the quadrotor body -->
+<!--     <xacro:include filename="$(find hector_sensors_description)/urdf/hokuyo_utm30lx.urdf.xacro" />
+    <xacro:hokuyo_utm30lx name="laser0" parent="base_link" ros_topic="scan" update_rate="40" ray_count="1081" min_angle="-135" max_angle="135">
+      <origin xyz="0.0 0.0 -0.097" rpy="${M_PI} 0 0"/>
+    </xacro:hokuyo_utm30lx> -->
     <xacro:include filename="$(find hector_sensors_description)/urdf/wireless_receiver.urdf.xacro" />
     <xacro:wireless_receiver name="wireless_receiver" parent="base_link" ros_topic="/wireless_receiver" update_rate="100">

File: hector_quadrotor_gazebo/urdf/quadrotor_sensors.gazebo.xacro (robot description, xacro)
@@ -12,12 +12,13 @@
             <rpyOffsets>0 0 0</rpyOffsets> <!-- deprecated -->
             <gaussianNoise>0</gaussianNoise>  <!-- deprecated -->
-            <accelDrift>0.5 0.5 0.5</accelDrift>
+<!--             <accelDrift>0.5 0.5 0.5</accelDrift>
             <accelGaussianNoise>0.35 0.35 0.3</accelGaussianNoise>
             <rateDrift>0.1 0.1 0.1</rateDrift>
-            <rateGaussianNoise>0.05 0.05 0.015</rateGaussianNoise>
-<!--             <accelDrift>0 0 0</accelDrift>
-            <accelGaussianNoise>0.35 0.35 0.3</accelGaussianNoise>
+            <rateGaussianNoise>0.05 0.05 0.015</rateGaussianNoise> -->
+            <!-- without noise version -->
+            <accelDrift>0 0 0</accelDrift>
+            <accelGaussianNoise>0.01 0.01 0.01</accelGaussianNoise>
             <rateDrift>0 0 0</rateDrift>
-            <rateGaussianNoise>0.05 0.05 0.015</rateGaussianNoise> -->
+            <rateGaussianNoise>0.01 0.01 0.01</rateGaussianNoise>
           </plugin>
           <plugin name="quadrotor_baro_sim" filename="libhector_gazebo_ros_baro.so">
