Commit message: update the rviz and launch file

File: hector_quadrotor_description/urdf/quadrotor_with_kinect.urdf.xacro (robot description, xacro)
@@ -9,5 +9,6 @@
     <xacro:include filename="$(find hector_sensors_description)/urdf/kinect_camera.urdf.xacro" />
     <xacro:kinect_camera name="camera" parent="base_link">
-      <origin xyz="0.05 0.0 -0.06" rpy="0 0 0"/>
+      <origin xyz="0.05 0.0 -0.06" rpy="0 ${M_PI/2} 0"/>
+      <!-- <origin xyz="0.05 0.0 -0.06" rpy="0 0 0"/> -->
     </xacro:kinect_camera>
 </robot>

File: hector_quadrotor_description/urdf/quadrotor_with_velodyne.urdf.xacro (robot description, xacro)
@@ -8,5 +8,5 @@
     <xacro:include filename="$(find velodyne_description)/urdf/VLP-16.urdf.xacro"/>
     <VLP-16 parent="base_link" name="velodyne" topic="/velodyne_points">
-    <origin xyz="0 0 0.03" rpy="0 0 0" />
+    <origin xyz="0 0 0.1" rpy="0 0 0" />
     </VLP-16>
 <!--     <xacro:include filename="$(find velodyne_description)/urdf/HDL-32E.urdf.xacro"/>
